File: KBD8X-MK2.kicad_pcb (KiCad board)
At the start: 2 copper layers, 343.7 x 118.3 mm, 347 parts, among them J1 AVR-ISP-6, Q1 DSS60601MZ4-13, SW1 SW_Push, SW2 SW_SPDT, SW3 SW_SPDT, U1 ATmega32U4-MU, U2 PRTR5V0U2X, Y1 16MHz

Commit message: Footprint updates top two rows
Footprints have been updated on the top two rows of the PCB to add Alps switch compatibility.
Parts:
- SW_#0_1: renamed from MX_#0_1; value MX-1U -> 1U; footprint MX_Alps_Hybrid:MXOnly-1U -> MX_Alps_Hybrid:MX-1U
- SW_#1: renamed from MX_#1; value MX-1U -> 1U; footprint MX_Alps_Hybrid:MXOnly-1U -> MX_Alps_Hybrid:MX-1U
- SW_#2: renamed from MX_#2; value MX-1U -> 1U; footprint MX_Alps_Hybrid:MXOnly-1U -> MX_Alps_Hybrid:MX-1U
- SW_#3: renamed from MX_#3; value MX-1U -> 1U; footprint MX_Alps_Hybrid:MXOnly-1U -> MX_Alps_Hybrid:MX-1U
- SW_#4: renamed from MX_#4; value MX-1U -> 1U; footprint MX_Alps_Hybrid:MXOnly-1U -> MX_Alps_Hybrid:MX-1U
- SW_#5: renamed from MX_#5; value MX-1U -> 1U; footprint MX_Alps_Hybrid:MXOnly-1U -> MX_Alps_Hybrid:MX-1U
- SW_#6: renamed from MX_#6; value MX-1U -> 1U; footprint MX_Alps_Hybrid:MXOnly-1U -> MX_Alps_Hybrid:MX-1U
- SW_#7: renamed from MX_#7; value MX-1U -> 1U; footprint MX_Alps_Hybrid:MXOnly-1U -> MX_Alps_Hybrid:MX-1U
- SW_#8: renamed from MX_#8; value MX-1U -> 1U; footprint MX_Alps_Hybrid:MXOnly-1U -> MX_Alps_Hybrid:MX-1U
- SW_#9: renamed from MX_#9; value MX-1U -> 1U; footprint MX_Alps_Hybrid:MXOnly-1U -> MX_Alps_Hybrid:MX-1U
- SW_-1: renamed from MX_-1; value MX-1U -> 1U; footprint MX_Alps_Hybrid:MXOnly-1U -> MX_Alps_Hybrid:MX-1U
- SW_BACK1: renamed from MX_BACK1; value MX-2U -> 2U; footprint MX_Alps_Hybrid:MXOnly-2U -> MX_Alps_Hybrid:MX-2U
- SW_BACK2: renamed from MX_BACK2; value MX-1U -> 1U; footprint MX_Alps_Hybrid:MXOnly-1U -> MX_Alps_Hybrid:MX-1U
- SW_ESC1: renamed from MX_ESC1; value MX-1U -> 1U; footprint MX_Alps_Hybrid:MXOnly-1U -> MX_Alps_Hybrid:MX-1U
- SW_FN1: renamed from MX_FN1; value MX-1U -> 1U; footprint MX_Alps_Hybrid:MXOnly-1U -> MX_Alps_Hybrid:MX-1U
- SW_FN10: renamed from MX_FN10; value MX-1U -> 1U; footprint MX_Alps_Hybrid:MXOnly-1U -> MX_Alps_Hybrid:MX-1U
- SW_FN11: renamed from MX_FN11; value MX-1U -> 1U; footprint MX_Alps_Hybrid:MXOnly-1U -> MX_Alps_Hybrid:MX-1U
- SW_FN12: renamed from MX_FN12; value MX-1U -> 1U; footprint MX_Alps_Hybrid:MXOnly-1U -> MX_Alps_Hybrid:MX-1U
- SW_FN2: renamed from MX_FN2; value MX-1U -> 1U; footprint MX_Alps_Hybrid:MXOnly-1U -> MX_Alps_Hybrid:MX-1U
- SW_FN3: renamed from MX_FN3; value MX-1U -> 1U; footprint MX_Alps_Hybrid:MXOnly-1U -> MX_Alps_Hybrid:MX-1U
- SW_FN4: renamed from MX_FN4; value MX-1U -> 1U; footprint MX_Alps_Hybrid:MXOnly-1U -> MX_Alps_Hybrid:MX-1U
- SW_FN5: renamed from MX_FN5; value MX-1U -> 1U; footprint MX_Alps_Hybrid:MXOnly-1U -> MX_Alps_Hybrid:MX-1U
- SW_FN6: renamed from MX_FN6; value MX-1U -> 1U; footprint MX_Alps_Hybrid:MXOnly-1U -> MX_Alps_Hybrid:MX-1U
- SW_FN7: renamed from MX_FN7; value MX-1U -> 1U; footprint MX_Alps_Hybrid:MXOnly-1U -> MX_Alps_Hybrid:MX-1U
- SW_FN8: renamed from MX_FN8; value MX-1U -> 1U; footprint MX_Alps_Hybrid:MXOnly-1U -> MX_Alps_Hybrid:MX-1U
- SW_FN9: renamed from MX_FN9; value MX-1U -> 1U; footprint MX_Alps_Hybrid:MXOnly-1U -> MX_Alps_Hybrid:MX-1U
- SW_HOME1: renamed from MX_HOME1; value MX-1U -> 1U; footprint MX_Alps_Hybrid:MXOnly-1U -> MX_Alps_Hybrid:MX-1U
- SW_INS1: renamed from MX_INS1; value MX-1U -> 1U; footprint MX_Alps_Hybrid:MXOnly-1U -> MX_Alps_Hybrid:MX-1U
- SW_PAUSE1: renamed from MX_PAUSE1; value MX-1U -> 1U; footprint MX_Alps_Hybrid:MXOnly-1U -> MX_Alps_Hybrid:MX-1U
- SW_PGUP1: renamed from MX_PGUP1; value MX-1U -> 1U; footprint MX_Alps_Hybrid:MXOnly-1U -> MX_Alps_Hybrid:MX-1U
- SW_PRINT1: renamed from MX_PRINT1; value MX-1U -> 1U; footprint MX_Alps_Hybrid:MXOnly-1U -> MX_Alps_Hybrid:MX-1U
- SW_SLOCK1: renamed from MX_SLOCK1; value MX-1U -> 1U; footprint MX_Alps_Hybrid:MXOnly-1U -> MX_Alps_Hybrid:MX-1U
- SW_`1: renamed from MX_`1; value MX-1U -> 1U; footprint MX_Alps_Hybrid:MXOnly-1U -> MX_Alps_Hybrid:MX-1U
Routing:
- net +5V: track 2658.4 -> 2667.9 mm
- net GND: track 1191.1 -> 1193.0 mm
- net Net-(D97-Pad2): track 11.5 -> 12.2 mm
- net Net-(D93-Pad2): track 11.5 -> 12.2 mm
- net Net-(D13-Pad2): track 11.5 -> 12.2 mm
- net Net-(D11-Pad2): track 11.5 -> 12.2 mm
- net Net-(D3-Pad2): track 11.5 -> 12.2 mm
- net Net-(D7-Pad2): track 11.5 -> 12.2 mm

Commit message: Additional row footprint update
Update of a row of footprints from MX only to Alps compatible.
Parts:
- SW_DEL1: renamed from MX_DEL1; value MX-1U -> 1U; footprint MX_Alps_Hybrid:MXOnly-1U -> MX_Alps_Hybrid:MX-1U
- SW_E1: renamed from MX_E1; value MX-1U -> 1U; footprint MX_Alps_Hybrid:MXOnly-1U -> MX_Alps_Hybrid:MX-1U
- SW_END1: renamed from MX_END1; value MX-1U -> 1U; footprint MX_Alps_Hybrid:MXOnly-1U -> MX_Alps_Hybrid:MX-1U
- SW_I1: renamed from MX_I1; value MX-1U -> 1U; footprint MX_Alps_Hybrid:MXOnly-1U -> MX_Alps_Hybrid:MX-1U
- SW_O1: renamed from MX_O1; value MX-1U -> 1U; footprint MX_Alps_Hybrid:MXOnly-1U -> MX_Alps_Hybrid:MX-1U
- SW_P1: renamed from MX_P1; value MX-1U -> 1U; footprint MX_Alps_Hybrid:MXOnly-1U -> MX_Alps_Hybrid:MX-1U
- SW_PGDN1: renamed from MX_PGDN1; value MX-1U -> 1U; footprint MX_Alps_Hybrid:MXOnly-1U -> MX_Alps_Hybrid:MX-1U
- SW_Q1: renamed from MX_Q1; value MX-1U -> 1U; footprint MX_Alps_Hybrid:MXOnly-1U -> MX_Alps_Hybrid:MX-1U
- SW_R1: renamed from MX_R1; value MX-1U -> 1U; footprint MX_Alps_Hybrid:MXOnly-1U -> MX_Alps_Hybrid:MX-1U
- SW_T1: renamed from MX_T1; value MX-1U -> 1U; footprint MX_Alps_Hybrid:MXOnly-1U -> MX_Alps_Hybrid:MX-1U
- SW_TAB1: renamed from MX_TAB1; value MX-1.5U -> 1.5U; footprint MX_Alps_Hybrid:MXOnly-1.5U -> MX_Alps_Hybrid:MX-1.5U
- SW_U1: renamed from MX_U1; value MX-1U -> 1U; footprint MX_Alps_Hybrid:MXOnly-1U -> MX_Alps_Hybrid:MX-1U
- SW_W1: renamed from MX_W1; value MX-1U -> 1U; footprint MX_Alps_Hybrid:MXOnly-1U -> MX_Alps_Hybrid:MX-1U
- SW_Y1: renamed from MX_Y1; value MX-1U -> 1U; footprint MX_Alps_Hybrid:MXOnly-1U -> MX_Alps_Hybrid:MX-1U
- SW_[1: renamed from MX_[1; value MX-1U -> 1U; footprint MX_Alps_Hybrid:MXOnly-1U -> MX_Alps_Hybrid:MX-1U
- SW_\1: renamed from MX_\1; value MX-1.5U -> 1.5U; footprint MX_Alps_Hybrid:MXOnly-1.5U -> MX_Alps_Hybrid:MX-1.5U
- SW_\2: renamed from MX_\2; value MX-1U -> 1U; footprint MX_Alps_Hybrid:MXOnly-1U -> MX_Alps_Hybrid:MX-1U
- SW_]1: renamed from MX_]1; value MX-1U -> 1U; footprint MX_Alps_Hybrid:MXOnly-1U -> MX_Alps_Hybrid:MX-1U
Routing:
- net +5V: track 2667.9 -> 2674.9 mm
- net COL4: track 605.9 -> 602.0 mm
- net COL5: track 467.6 -> 463.8 mm
- net COL3: track 817.5 -> 815.6 mm
- net COL2: track 665.0 -> 663.1 mm
- net COL1: track 576.7 -> 574.8 mm
- net COL6: track 393.4 -> 391.7 mm
- net Net-(D48-Pad2): track 37.5 -> 38.4 mm
- net ROW6: track 357.3 -> 358.1 mm

Commit message: Additional row of footprint updates
Enter row footprints updated to Alps compatible.
Parts:
- SW_'1: renamed from MX_'1; value MX-1U -> 1U; footprint MX_Alps_Hybrid:MXOnly-1U -> MX_Alps_Hybrid:MX-1U
- SW_;1: renamed from MX_;1; value MX-1U -> 1U; footprint MX_Alps_Hybrid:MXOnly-1U -> MX_Alps_Hybrid:MX-1U
- SW_A1: renamed from MX_A1; value MX-1U -> 1U; footprint MX_Alps_Hybrid:MXOnly-1U -> MX_Alps_Hybrid:MX-1U
- SW_BACK3: renamed from MX_BACK3; value MX-1U -> 1U; footprint MX_Alps_Hybrid:MXOnly-1U -> MX_Alps_Hybrid:MX-1U
- SW_CLOCK1: renamed from MX_CLOCK1; value MX-1.75U -> 1.75U; footprint MX_Alps_Hybrid:MXOnly-1.75U -> MX_Alps_Hybrid:MX-1.75U
- SW_CLOCK2: renamed from MX_CLOCK2; value MX-1.25U -> 1.25U; footprint MX_Alps_Hybrid:MXOnly-1.25U-FLIPPED -> MX_Alps_Hybrid:MX-1.25U-FLIPPED
- SW_D1: renamed from MX_D1; value MX-1U -> 1U; footprint MX_Alps_Hybrid:MXOnly-1U -> MX_Alps_Hybrid:MX-1U
- SW_F1: renamed from MX_F1; value MX-1U -> 1U; footprint MX_Alps_Hybrid:MXOnly-1U -> MX_Alps_Hybrid:MX-1U
- SW_G1: renamed from MX_G1; value MX-1U -> 1U; footprint MX_Alps_Hybrid:MXOnly-1U -> MX_Alps_Hybrid:MX-1U
- SW_H1: renamed from MX_H1; value MX-1U -> 1U; footprint MX_Alps_Hybrid:MXOnly-1U -> MX_Alps_Hybrid:MX-1U
- SW_J1: renamed from MX_J1; value MX-1U -> 1U; footprint MX_Alps_Hybrid:MXOnly-1U -> MX_Alps_Hybrid:MX-1U
- SW_K1: renamed from MX_K1; value MX-1U -> 1U; footprint MX_Alps_Hybrid:MXOnly-1U -> MX_Alps_Hybrid:MX-1U
- SW_L1: renamed from MX_L1; value MX-1U -> 1U; footprint MX_Alps_Hybrid:MXOnly-1U -> MX_Alps_Hybrid:MX-1U
- SW_RETURN1: renamed from MX_RETURN1; value MX-2.25U -> 2.25U; footprint MX_Alps_Hybrid:MXOnly-2.25U -> MX_Alps_Hybrid:MX-2.25U
- SW_RETURN2: renamed from MX_RETURN2; value MX-ISO -> ISO; footprint MX_Alps_Hybrid:MXOnly-ISO-ROTATED-ReversedStabilizers -> MX_Alps_Hybrid:MX-ISO-ReversedStabilizers
- SW_S1: renamed from MX_S1; value MX-1U -> 1U; footprint MX_Alps_Hybrid:MXOnly-1U -> MX_Alps_Hybrid:MX-1U
Routing:
- net +5V: track 2674.9 -> 2713.4 mm
- net Net-(D65-Pad2): track 41.0 -> 42.1 mm
- net Net-(D101-Pad2): track 11.5 -> 12.5 mm

Commit message: Additional footprint updates
Parts:
- SW_,1: renamed from MX_,1; value MX-1U -> 1U; footprint MX_Alps_Hybrid:MXOnly-1U -> MX_Alps_Hybrid:MX-1U
- SW_.1: renamed from MX_.1; value MX-1U -> 1U; footprint MX_Alps_Hybrid:MXOnly-1U -> MX_Alps_Hybrid:MX-1U
- SW_/1: renamed from MX_/1; value MX-1U -> 1U; footprint MX_Alps_Hybrid:MXOnly-1U -> MX_Alps_Hybrid:MX-1U
- SW_B1: renamed from MX_B1; value MX-1U -> 1U; footprint MX_Alps_Hybrid:MXOnly-1U -> MX_Alps_Hybrid:MX-1U
- SW_C1: renamed from MX_C1; value MX-1U -> 1U; footprint MX_Alps_Hybrid:MXOnly-1U -> MX_Alps_Hybrid:MX-1U
- SW_LSHIFT1: renamed from MX_LSHIFT1; value MX-2.25U -> 2.25U; footprint MX_Alps_Hybrid:MXOnly-2.25U -> MX_Alps_Hybrid:MX-2.25U
- SW_LSHIFT2: renamed from MX_LSHIFT2; value MX-1.25U -> 1.25U; footprint MX_Alps_Hybrid:MXOnly-1.25U -> MX_Alps_Hybrid:MX-1.25U
- SW_LSHIFT3: renamed from MX_LSHIFT3; value MX-1U -> 1U; footprint MX_Alps_Hybrid:MXOnly-1U -> MX_Alps_Hybrid:MX-1U
- SW_M1: renamed from MX_M1; value MX-1U -> 1U; footprint MX_Alps_Hybrid:MXOnly-1U -> MX_Alps_Hybrid:MX-1U
- SW_N1: renamed from MX_N1; value MX-1U -> 1U; footprint MX_Alps_Hybrid:MXOnly-1U -> MX_Alps_Hybrid:MX-1U
- SW_RSHIFT1: renamed from MX_RSHIFT1; value MX-2.75U -> 2.75U; footprint MX_Alps_Hybrid:MXOnly-2.75U -> MX_Alps_Hybrid:MX-2.75U
- SW_RSHIFT2: renamed from MX_RSHIFT2; value MX-1.75U -> 1.75U; footprint MX_Alps_Hybrid:MXOnly-1.75U -> MX_Alps_Hybrid:MX-1.75U
- SW_RSHIFT3: renamed from MX_RSHIFT3; value MX-1U -> 1U; footprint MX_Alps_Hybrid:MXOnly-1U -> MX_Alps_Hybrid:MX-1U
- SW_UP1: renamed from MX_UP1; value MX-1U -> 1U; footprint MX_Alps_Hybrid:MXOnly-1U -> MX_Alps_Hybrid:MX-1U
- SW_V1: renamed from MX_V1; value MX-1U -> 1U; footprint MX_Alps_Hybrid:MXOnly-1U -> MX_Alps_Hybrid:MX-1U
- SW_X1: renamed from MX_X1; value MX-1U -> 1U; footprint MX_Alps_Hybrid:MXOnly-1U -> MX_Alps_Hybrid:MX-1U
- SW_Z1: renamed from MX_Z1; value MX-1U -> 1U; footprint MX_Alps_Hybrid:MXOnly-1U -> MX_Alps_Hybrid:MX-1U
Routing:
- net COL4: track 602.0 -> 598.2 mm
- net COL5: track 463.8 -> 460.0 mm
- net +5V: track 2713.4 -> 2710.2 mm
- net COL1: track 574.8 -> 572.9 mm
- net COL2: track 663.1 -> 661.1 mm
- net COL3: track 815.6 -> 813.7 mm
- net Net-(D67-Pad2): track 35.7 -> 37.0 mm
- net Net-(D78-Pad2): track 16.0 -> 17.2 mm

Commit message: Final footprint updates
All rows have been updated to Alps compatible switch footprints.
Parts:
- SW_DN1: renamed from MX_DN1; value MX-1U -> 1U; footprint MX_Alps_Hybrid:MXOnly-1U -> MX_Alps_Hybrid:MX-1U
- SW_LALT1: renamed from MX_LALT1; value MX-1.25U -> 1.25U; footprint MX_Alps_Hybrid:MXOnly-1.25U -> MX_Alps_Hybrid:MX-1.25U
- SW_LALT2: renamed from MX_LALT2; value MX-1.5U -> 1.5U; footprint MX_Alps_Hybrid:MXOnly-1.5U-FLIPPED -> MX_Alps_Hybrid:MX-1.5U-FLIPPED
- SW_LCTRL1: renamed from MX_LCTRL1; value MX-1.25U -> 1.25U; footprint MX_Alps_Hybrid:MXOnly-1.25U -> MX_Alps_Hybrid:MX-1.25U
- SW_LCTRL2: renamed from MX_LCTRL2; value MX-1.5U -> 1.5U; footprint MX_Alps_Hybrid:MXOnly-1.5U-FLIPPED -> MX_Alps_Hybrid:MX-1.5U-FLIPPED
- SW_LFT1: renamed from MX_LFT1; value MX-1U -> 1U; footprint MX_Alps_Hybrid:MXOnly-1U -> MX_Alps_Hybrid:MX-1U
- SW_LGUI1: renamed from MX_LGUI1; value MX-1.25U -> 1.25U; footprint MX_Alps_Hybrid:MXOnly-1.25U -> MX_Alps_Hybrid:MX-1.25U
- SW_LGUI2: renamed from MX_LGUI2; value MX-1U -> 1U; footprint MX_Alps_Hybrid:MXOnly-1U-FLIPPED -> MX_Alps_Hybrid:MX-1U-FLIPPED
- SW_RALT1: renamed from MX_RALT1; value MX-1.25U -> 1.25U; footprint MX_Alps_Hybrid:MXOnly-1.25U -> MX_Alps_Hybrid:MX-1.25U
- SW_RALT2: renamed from MX_RALT2; value MX-1.5U -> 1.5U; footprint MX_Alps_Hybrid:MXOnly-1.5U -> MX_Alps_Hybrid:MX-1.5U
- SW_RCTRL1: renamed from MX_RCTRL1; value MX-1.25U -> 1.25U; footprint MX_Alps_Hybrid:MXOnly-1.25U-FLIPPED -> MX_Alps_Hybrid:MX-1.25U-FLIPPED
- SW_RCTRL2: renamed from MX_RCTRL2; value MX-1.5U -> 1.5U; footprint MX_Alps_Hybrid:MXOnly-1.5U -> MX_Alps_Hybrid:MX-1.5U
- SW_RGUI1: renamed from MX_RGUI1; value MX-1.25U -> 1.25U; footprint MX_Alps_Hybrid:MXOnly-1.25U-FLIPPED -> MX_Alps_Hybrid:MX-1.25U-FLIPPED
- SW_RGUI2: renamed from MX_RGUI2; value MX-1U -> 1U; footprint MX_Alps_Hybrid:MXOnly-1U -> MX_Alps_Hybrid:MX-1U
- SW_RMENU1: renamed from MX_RMENU1; footprint MX_Alps_Hybrid:MXOnly-1.25U-FLIPPED -> MX_Alps_Hybrid:MX-1.25U-FLIPPED
- SW_RT1: renamed from MX_RT1; value MX-1U -> 1U; footprint MX_Alps_Hybrid:MXOnly-1U -> MX_Alps_Hybrid:MX-1U
- SW_SP1: renamed from MX_SP1; value MX-6.25U -> 6.25U; footprint MX_Alps_Hybrid:MXOnly-6.25U-ReversedStabilizers -> MX_Alps_Hybrid:MX-6.25U-ReversedStabilizers
- SW_SP2: renamed from MX_SP2; value MX-7U -> 7U; footprint MX_Alps_Hybrid:MXOnly-7U-ReversedStabilizers -> MX_Alps_Hybrid:MX-7U-ReversedStabilizers
Routing:
- net +5V: track 2710.2 -> 2712.9 mm
- net GND: track 1193.0 -> 1195.1 mm
- net COL5: track 460.0 -> 458.5 mm
- net Net-(D111-Pad2): track 11.5 -> 12.5 mm
- net Net-(D86-Pad2): track 13.9 -> 14.7 mm
- net Net-(D82-Pad2): track 13.9 -> 14.7 mm
- net Net-(D91-Pad2): track 13.9 -> 14.6 mm
Other:
- board text added: "Alps modifications by robotictomato"
- board text added: "KBD8X-MKII PCB Rev 2.1 20211124"
- board text removed: "KBD8X-MKII PCB Rev 2.0 20190404"
