File: matrix.sch (KiCad schematic (older format))
At the start: 285 parts, among them SW2 SW_SPDT, SW3 SW_SPDT

Commit message: Additional footprint updates
Parts:
- SW_,1: renamed from MX_,1; value MX-1U -> 1U; footprint MX_Alps_Hybrid:MXOnly-1U -> MX_Alps_Hybrid:MX-1U
- SW_.1: renamed from MX_.1; value MX-1U -> 1U; footprint MX_Alps_Hybrid:MXOnly-1U -> MX_Alps_Hybrid:MX-1U
- SW_/1: renamed from MX_/1; value MX-1U -> 1U; footprint MX_Alps_Hybrid:MXOnly-1U -> MX_Alps_Hybrid:MX-1U
- SW_B1: renamed from MX_B1; value MX-1U -> 1U; footprint MX_Alps_Hybrid:MXOnly-1U -> MX_Alps_Hybrid:MX-1U
- SW_C1: renamed from MX_C1; value MX-1U -> 1U; footprint MX_Alps_Hybrid:MXOnly-1U -> MX_Alps_Hybrid:MX-1U
- SW_LSHIFT1: renamed from MX_LSHIFT1; value MX-2.25U -> 2.25U; footprint MX_Alps_Hybrid:MXOnly-2.25U -> MX_Alps_Hybrid:MX-2.25U
- SW_LSHIFT2: renamed from MX_LSHIFT2; value MX-1.25U -> 1.25U; footprint MX_Alps_Hybrid:MXOnly-1.25U -> MX_Alps_Hybrid:MX-1.25U
- SW_LSHIFT3: renamed from MX_LSHIFT3; value MX-1U -> 1U; footprint MX_Alps_Hybrid:MXOnly-1U -> MX_Alps_Hybrid:MX-1U
- SW_M1: renamed from MX_M1; value MX-1U -> 1U; footprint MX_Alps_Hybrid:MXOnly-1U -> MX_Alps_Hybrid:MX-1U
- SW_N1: renamed from MX_N1; value MX-1U -> 1U; footprint MX_Alps_Hybrid:MXOnly-1U -> MX_Alps_Hybrid:MX-1U
- SW_RSHIFT1: renamed from MX_RSHIFT1; value MX-2.75U -> 2.75U; footprint MX_Alps_Hybrid:MXOnly-2.75U -> MX_Alps_Hybrid:MX-2.75U
- SW_RSHIFT2: renamed from MX_RSHIFT2; value MX-1.75U -> 1.75U; footprint MX_Alps_Hybrid:MXOnly-1.75U -> MX_Alps_Hybrid:MX-1.75U
- SW_RSHIFT3: renamed from MX_RSHIFT3; value MX-1U -> 1U; footprint MX_Alps_Hybrid:MXOnly-1U -> MX_Alps_Hybrid:MX-1U
- SW_UP1: renamed from MX_UP1; value MX-1U -> 1U; footprint MX_Alps_Hybrid:MXOnly-1U -> MX_Alps_Hybrid:MX-1U
- SW_V1: renamed from MX_V1; value MX-1U -> 1U; footprint MX_Alps_Hybrid:MXOnly-1U -> MX_Alps_Hybrid:MX-1U
- SW_X1: renamed from MX_X1; value MX-1U -> 1U; footprint MX_Alps_Hybrid:MXOnly-1U -> MX_Alps_Hybrid:MX-1U
- SW_Z1: renamed from MX_Z1; value MX-1U -> 1U; footprint MX_Alps_Hybrid:MXOnly-1U -> MX_Alps_Hybrid:MX-1U
Changed lines of the file:
@@
 $EndComp
 $Comp
-L MX_Alps_Hybrids:MX-2.25U MX_LSHIFT1
+L MX_Alps_Hybrids:MX-2.25U SW_LSHIFT1
 U 1 1 5A2F4AA7
 P 4825 5450
-F 0 "MX_LSHIFT1" H 4825 5575 60  0000 C CNN
-F 1 "MX-2.25U" H 4825 5500 20  0000 C CNN
-F 2 "MX_Alps_Hybrid:MXOnly-2.25U" H 4800 5425 60  0001 C CNN
+F 0 "SW_LSHIFT1" H 4825 5575 60  0000 C CNN
+F 1 "2.25U" H 4825 5500 20  0000 C CNN
+F 2 "MX_Alps_Hybrid:MX-2.25U" H 4800 5425 60  0001 C CNN
 F 3 "" H 4800 5425 60  0001 C CNN
 	1    4825 5450
@@
 $EndComp
 $Comp
-L MX_Alps_Hybrids:MX-1U MX_X1
+L MX_Alps_Hybrids:MX-1U SW_X1
 U 1 1 5A2F4ACF
 P 6700 5450
-F 0 "MX_X1" H 6700 5575 60  0000 C CNN
-F 1 "MX-1U" H 6700 5500 20  0000 C CNN
-F 2 "MX_Alps_Hybrid:MXOnly-1U" H 6675 5425 60  0001 C CNN
+F 0 "SW_X1" H 6700 5575 60  0000 C CNN
+F 1 "1U" H 6700 5500 20  0000 C CNN
+F 2 "MX_Alps_Hybrid:MX-1U" H 6675 5425 60  0001 C CNN
 F 3 "" H 6675 5425 60  0001 C CNN
 	1    6700 5450
@@
 $EndComp
 $Comp
-L MX_Alps_Hybrids:MX-1U MX_C1
+L MX_Alps_Hybrids:MX-1U SW_C1
 U 1 1 5A2F4AE3
 P 7325 5450
-F 0 "MX_C1" H 7325 5575 60  0000 C CNN
-F 1 "MX-1U" H 7325 5500 20  0000 C CNN
-F 2 "MX_Alps_Hybrid:MXOnly-1U" H 7300 5425 60  0001 C CNN
+F 0 "SW_C1" H 7325 5575 60  0000 C CNN
+F 1 "1U" H 7325 5500 20  0000 C CNN
+F 2 "MX_Alps_Hybrid:MX-1U" H 7300 5425 60  0001 C CNN
 F 3 "" H 7300 5425 60  0001 C CNN
 	1    7325 5450
@@
 $EndComp
 $Comp
-L MX_Alps_Hybrids:MX-1U MX_V1
+L MX_Alps_Hybrids:MX-1U SW_V1
 U 1 1 5A2F4AF7
 P 7950 5450
-F 0 "MX_V1" H 7950 5575 60  0000 C CNN
-F 1 "MX-1U" H 7950 5500 20  0000 C CNN
-F 2 "MX_Alps_Hybrid:MXOnly-1U" H 7925 5425 60  0001 C CNN
+F 0 "SW_V1" H 7950 5575 60  0000 C CNN
+F 1 "1U" H 7950 5500 20  0000 C CNN
+F 2 "MX_Alps_Hybrid:MX-1U" H 7925 5425 60  0001 C CNN
 F 3 "" H 7925 5425 60  0001 C CNN
 	1    7950 5450
@@
 $EndComp
 $Comp
-L MX_Alps_Hybrids:MX-1U MX_B1
+L MX_Alps_Hybrids:MX-1U SW_B1
 U 1 1 5A2F4B0B
 P 8575 5450
-F 0 "MX_B1" H 8575 5575 60  0000 C CNN
-F 1 "MX-1U" H 8575 5500 20  0000 C CNN
-F 2 "MX_Alps_Hybrid:MXOnly-1U" H 8550 5425 60  0001 C CNN
+F 0 "SW_B1" H 8575 5575 60  0000 C CNN
+F 1 "1U" H 8575 5500 20  0000 C CNN
+F 2 "MX_Alps_Hybrid:MX-1U" H 8550 5425 60  0001 C CNN
 F 3 "" H 8550 5425 60  0001 C CNN
 	1    8575 5450
@@
 $EndComp
 $Comp
-L MX_Alps_Hybrids:MX-1U MX_N1
+L MX_Alps_Hybrids:MX-1U SW_N1
 U 1 1 5A2F4B1F
 P 9200 5450
-F 0 "MX_N1" H 9200 5575 60  0000 C CNN
-F 1 "MX-1U" H 9200 5500 20  0000 C CNN
-F 2 "MX_Alps_Hybrid:MXOnly-1U" H 9175 5425 60  0001 C CNN
+F 0 "SW_N1" H 9200 5575 60  0000 C CNN
+F 1 "1U" H 9200 5500 20  0000 C CNN
+F 2 "MX_Alps_Hybrid:MX-1U" H 9175 5425 60  0001 C CNN
 F 3 "" H 9175 5425 60  0001 C CNN
 	1    9200 5450
@@
 $EndComp
 $Comp
-L MX_Alps_Hybrids:MX-1U MX_M1
+L MX_Alps_Hybrids:MX-1U SW_M1
 U 1 1 5A2F4B33
 P 9825 5450
-F 0 "MX_M1" H 9825 5575 60  0000 C CNN
-F 1 "MX-1U" H 9825 5500 20  0000 C CNN
-F 2 "MX_Alps_Hybrid:MXOnly-1U" H 9800 5425 60  0001 C CNN
+F 0 "SW_M1" H 9825 5575 60  0000 C CNN
+F 1 "1U" H 9825 5500 20  0000 C CNN
+F 2 "MX_Alps_Hybrid:MX-1U" H 9800 5425 60  0001 C CNN
 F 3 "" H 9800 5425 60  0001 C CNN
 	1    9825 5450
@@
 $EndComp
 $Comp
-L MX_Alps_Hybrids:MX-1U MX_,1
+L MX_Alps_Hybrids:MX-1U SW_,1
 U 1 1 5A2F4B47
 P 10450 5450
-F 0 "MX_,1" H 10450 5575 60  0000 C CNN
-F 1 "MX-1U" H 10450 5500 20  0000 C CNN
-F 2 "MX_Alps_Hybrid:MXOnly-1U" H 10425 5425 60  0001 C CNN
+F 0 "SW_,1" H 10450 5575 60  0000 C CNN
+F 1 "1U" H 10450 5500 20  0000 C CNN
+F 2 "MX_Alps_Hybrid:MX-1U" H 10425 5425 60  0001 C CNN
 F 3 "" H 10425 5425 60  0001 C CNN
 	1    10450 5450
@@
 $EndComp
 $Comp
-L MX_Alps_Hybrids:MX-1U MX_.1
+L MX_Alps_Hybrids:MX-1U SW_.1
 U 1 1 5A2F4B5B
 P 11075 5450
-F 0 "MX_.1" H 11075 5575 60  0000 C CNN
-F 1 "MX-1U" H 11075 5500 20  0000 C CNN
-F 2 "MX_Alps_Hybrid:MXOnly-1U" H 11050 5425 60  0001 C CNN
+F 0 "SW_.1" H 11075 5575 60  0000 C CNN
+F 1 "1U" H 11075 5500 20  0000 C CNN
+F 2 "MX_Alps_Hybrid:MX-1U" H 11050 5425 60  0001 C CNN
 F 3 "" H 11050 5425 60  0001 C CNN
 	1    11075 5450
@@
 $EndComp
 $Comp
-L MX_Alps_Hybrids:MX-1U MX_/1
+L MX_Alps_Hybrids:MX-1U SW_/1
 U 1 1 5A2F4B6F
 P 11700 5450
-F 0 "MX_/1" H 11700 5575 60  0000 C CNN
-F 1 "MX-1U" H 11700 5500 20  0000 C CNN
-F 2 "MX_Alps_Hybrid:MXOnly-1U" H 11675 5425 60  0001 C CNN
+F 0 "SW_/1" H 11700 5575 60  0000 C CNN
+F 1 "1U" H 11700 5500 20  0000 C CNN
+F 2 "MX_Alps_Hybrid:MX-1U" H 11675 5425 60  0001 C CNN
 F 3 "" H 11675 5425 60  0001 C CNN
 	1    11700 5450
@@
 $EndComp
 $Comp
-L MX_Alps_Hybrids:MX-1U MX_RSHIFT1
+L MX_Alps_Hybrids:MX-1U SW_RSHIFT1
 U 1 1 5A2F4B83
 P 12325 5450
-F 0 "MX_RSHIFT1" H 12325 5575 60  0000 C CNN
-F 1 "MX-2.75U" H 12325 5500 20  0000 C CNN
-F 2 "MX_Alps_Hybrid:MXOnly-2.75U" H 12300 5425 60  0001 C CNN
+F 0 "SW_RSHIFT1" H 12325 5575 60  0000 C CNN
+F 1 "2.75U" H 12325 5500 20  0000 C CNN
+F 2 "MX_Alps_Hybrid:MX-2.75U" H 12300 5425 60  0001 C CNN
 F 3 "" H 12300 5425 60  0001 C CNN
 	1    12325 5450
@@
 $EndComp
 $Comp
-L MX_Alps_Hybrids:MX-1U MX_Z1
+L MX_Alps_Hybrids:MX-1U SW_Z1
 U 1 1 5A2F4ABB
 P 6075 5450
-F 0 "MX_Z1" H 6075 5575 60  0000 C CNN
-F 1 "MX-1U" H 6075 5500 20  0000 C CNN
-F 2 "MX_Alps_Hybrid:MXOnly-1U" H 6050 5425 60  0001 C CNN
+F 0 "SW_Z1" H 6075 5575 60  0000 C CNN
+F 1 "1U" H 6075 5500 20  0000 C CNN
+F 2 "MX_Alps_Hybrid:MX-1U" H 6050 5425 60  0001 C CNN
 F 3 "" H 6050 5425 60  0001 C CNN
 	1    6075 5450
@@
 $EndComp
 $Comp
-L MX_Alps_Hybrids:MX-1U MX_RSHIFT3
+L MX_Alps_Hybrids:MX-1U SW_RSHIFT3
 U 1 1 5A2F4BE7
 P 12950 5450
-F 0 "MX_RSHIFT3" H 12950 5575 60  0000 C CNN
-F 1 "MX-1U" H 12950 5500 20  0000 C CNN
-F 2 "MX_Alps_Hybrid:MXOnly-1U" H 12925 5425 60  0001 C CNN
+F 0 "SW_RSHIFT3" H 12950 5575 60  0000 C CNN
+F 1 "1U" H 12950 5500 20  0000 C CNN
+F 2 "MX_Alps_Hybrid:MX-1U" H 12925 5425 60  0001 C CNN
 F 3 "" H 12925 5425 60  0001 C CNN
 	1    12950 5450
@@
 Connection ~ 16325 5475
 $Comp
-L MX_Alps_Hybrids:MX-1U MX_UP1
+L MX_Alps_Hybrids:MX-1U SW_UP1
 U 1 1 5ADCFAD2
 P 16200 5450
-F 0 "MX_UP1" H 16200 5575 60  0000 C CNN
-F 1 "MX-1U" H 16200 5500 20  0000 C CNN
-F 2 "MX_Alps_Hybrid:MXOnly-1U" H 16175 5425 60  0001 C CNN
+F 0 "SW_UP1" H 16200 5575 60  0000 C CNN
+F 1 "1U" H 16200 5500 20  0000 C CNN
+F 2 "MX_Alps_Hybrid:MX-1U" H 16175 5425 60  0001 C CNN
 F 3 "" H 16175 5425 60  0001 C CNN
 	1    16200 5450
@@
 $EndComp
 $Comp
-L MX_Alps_Hybrids:MX-1U MX_LSHIFT3
+L MX_Alps_Hybrids:MX-1U SW_LSHIFT3
 U 1 1 5DD5E02C
 P 5450 5450
-F 0 "MX_LSHIFT3" H 5450 5575 60  0000 C CNN
-F 1 "MX-1U" H 5450 5500 20  0000 C CNN
-F 2 "MX_Alps_Hybrid:MXOnly-1U" H 5425 5425 60  0001 C CNN
+F 0 "SW_LSHIFT3" H 5450 5575 60  0000 C CNN
+F 1 "1U" H 5450 5500 20  0000 C CNN
+F 2 "MX_Alps_Hybrid:MX-1U" H 5425 5425 60  0001 C CNN
 F 3 "" H 5425 5425 60  0001 C CNN
 	1    5450 5450
@@
 Connection ~ 5775 4750
 $Comp
-L MX_Alps_Hybrids:MX-2.25U MX_LSHIFT2
+L MX_Alps_Hybrids:MX-2.25U SW_LSHIFT2
 U 1 1 5DF0DCEF
 P 4250 5450
-F 0 "MX_LSHIFT2" H 4250 5575 60  0000 C CNN
-F 1 "MX-1.25U" H 4250 5500 20  0000 C CNN
-F 2 "MX_Alps_Hybrid:MXOnly-1.25U" H 4225 5425 60  0001 C CNN
+F 0 "SW_LSHIFT2" H 4250 5575 60  0000 C CNN
+F 1 "1.25U" H 4250 5500 20  0000 C CNN
+F 2 "MX_Alps_Hybrid:MX-1.25U" H 4225 5425 60  0001 C CNN
 F 3 "" H 4225 5425 60  0001 C CNN
 	1    4250 5450
@@
 	8675 6600 11175 6600
 $Comp
-L MX_Alps_Hybrids:MX-1U MX_RSHIFT2
+L MX_Alps_Hybrids:MX-1U SW_RSHIFT2
 U 1 1 5F321443
 P 13675 5450
-F 0 "MX_RSHIFT2" H 13675 5575 60  0000 C CNN
-F 1 "MX-1.75U" H 13675 5500 20  0000 C CNN
-F 2 "MX_Alps_Hybrid:MXOnly-1.75U" H 13650 5425 60  0001 C CNN
+F 0 "SW_RSHIFT2" H 13675 5575 60  0000 C CNN
+F 1 "1.75U" H 13675 5500 20  0000 C CNN
+F 2 "MX_Alps_Hybrid:MX-1.75U" H 13650 5425 60  0001 C CNN
 F 3 "" H 13650 5425 60  0001 C CNN
 	1    13675 5450

Commit message: Final footprint updates
All rows have been updated to Alps compatible switch footprints.
Parts:
- SW_DN1: renamed from MX_DN1; value MX-1U -> 1U; footprint MX_Alps_Hybrid:MXOnly-1U -> MX_Alps_Hybrid:MX-1U
- SW_LALT1: renamed from MX_LALT1; value MX-1.25U -> 1.25U; footprint MX_Alps_Hybrid:MXOnly-1.25U -> MX_Alps_Hybrid:MX-1.25U
- SW_LALT2: renamed from MX_LALT2; value MX-1.5U -> 1.5U; footprint MX_Alps_Hybrid:MXOnly-1.5U-FLIPPED -> MX_Alps_Hybrid:MX-1.5U-FLIPPED
- SW_LCTRL1: renamed from MX_LCTRL1; value MX-1.25U -> 1.25U; footprint MX_Alps_Hybrid:MXOnly-1.25U -> MX_Alps_Hybrid:MX-1.25U
- SW_LCTRL2: renamed from MX_LCTRL2; value MX-1.5U -> 1.5U; footprint MX_Alps_Hybrid:MXOnly-1.5U-FLIPPED -> MX_Alps_Hybrid:MX-1.5U-FLIPPED
- SW_LFT1: renamed from MX_LFT1; value MX-1U -> 1U; footprint MX_Alps_Hybrid:MXOnly-1U -> MX_Alps_Hybrid:MX-1U
- SW_LGUI1: renamed from MX_LGUI1; value MX-1.25U -> 1.25U; footprint MX_Alps_Hybrid:MXOnly-1.25U -> MX_Alps_Hybrid:MX-1.25U
- SW_LGUI2: renamed from MX_LGUI2; value MX-1U -> 1U; footprint MX_Alps_Hybrid:MXOnly-1U-FLIPPED -> MX_Alps_Hybrid:MX-1U-FLIPPED
- SW_RALT1: renamed from MX_RALT1; value MX-1.25U -> 1.25U; footprint MX_Alps_Hybrid:MXOnly-1.25U -> MX_Alps_Hybrid:MX-1.25U
- SW_RALT2: renamed from MX_RALT2; value MX-1.5U -> 1.5U; footprint MX_Alps_Hybrid:MXOnly-1.5U -> MX_Alps_Hybrid:MX-1.5U
- SW_RCTRL1: renamed from MX_RCTRL1; value MX-1.25U -> 1.25U; footprint MX_Alps_Hybrid:MXOnly-1.25U-FLIPPED -> MX_Alps_Hybrid:MX-1.25U-FLIPPED
- SW_RCTRL2: renamed from MX_RCTRL2; value MX-1.5U -> 1.5U; footprint MX_Alps_Hybrid:MXOnly-1.5U -> MX_Alps_Hybrid:MX-1.5U
- SW_RGUI1: renamed from MX_RGUI1; value MX-1.25U -> 1.25U; footprint MX_Alps_Hybrid:MXOnly-1.25U-FLIPPED -> MX_Alps_Hybrid:MX-1.25U-FLIPPED
- SW_RGUI2: renamed from MX_RGUI2; value MX-1U -> 1U; footprint MX_Alps_Hybrid:MXOnly-1U -> MX_Alps_Hybrid:MX-1U
- SW_RMENU1: renamed from MX_RMENU1; footprint MX_Alps_Hybrid:MXOnly-1.25U-FLIPPED -> MX_Alps_Hybrid:MX-1.25U-FLIPPED
- SW_RT1: renamed from MX_RT1; value MX-1U -> 1U; footprint MX_Alps_Hybrid:MXOnly-1U -> MX_Alps_Hybrid:MX-1U
- SW_SP1: renamed from MX_SP1; value MX-6.25U -> 6.25U; footprint MX_Alps_Hybrid:MXOnly-6.25U-ReversedStabilizers -> MX_Alps_Hybrid:MX-6.25U-ReversedStabilizers
- SW_SP2: renamed from MX_SP2; value MX-7U -> 7U; footprint MX_Alps_Hybrid:MXOnly-7U-ReversedStabilizers -> MX_Alps_Hybrid:MX-7U-ReversedStabilizers
Changed lines of the file:
@@
 $EndComp
 $Comp
-L MX_Alps_Hybrids:MX-1U MX_LCTRL1
+L MX_Alps_Hybrids:MX-1U SW_LCTRL1
 U 1 1 5A2F4C0F
 P 4825 6125
-F 0 "MX_LCTRL1" H 4825 6250 60  0000 C CNN
-F 1 "MX-1.25U" H 4825 6175 20  0000 C CNN
-F 2 "MX_Alps_Hybrid:MXOnly-1.25U" H 4800 6100 60  0001 C CNN
+F 0 "SW_LCTRL1" H 4825 6250 60  0000 C CNN
+F 1 "1.25U" H 4825 6175 20  0000 C CNN
+F 2 "MX_Alps_Hybrid:MX-1.25U" H 4800 6100 60  0001 C CNN
 F 3 "" H 4800 6100 60  0001 C CNN
 	1    4825 6125
@@
 $EndComp
 $Comp
-L MX_Alps_Hybrids:MX-1.25U MX_LGUI1
+L MX_Alps_Hybrids:MX-1.25U SW_LGUI1
 U 1 1 5A2F4C23
 P 5450 6125
-F 0 "MX_LGUI1" H 5450 6250 60  0000 C CNN
-F 1 "MX-1.25U" H 5450 6175 20  0000 C CNN
-F 2 "MX_Alps_Hybrid:MXOnly-1.25U" H 5425 6100 60  0001 C CNN
+F 0 "SW_LGUI1" H 5450 6250 60  0000 C CNN
+F 1 "1.25U" H 5450 6175 20  0000 C CNN
+F 2 "MX_Alps_Hybrid:MX-1.25U" H 5425 6100 60  0001 C CNN
 F 3 "" H 5425 6100 60  0001 C CNN
 	1    5450 6125
@@
 $EndComp
 $Comp
-L MX_Alps_Hybrids:MX-1.25U MX_LALT1
+L MX_Alps_Hybrids:MX-1.25U SW_LALT1
 U 1 1 5A2F4C37
 P 6075 6125
-F 0 "MX_LALT1" H 6075 6250 60  0000 C CNN
-F 1 "MX-1.25U" H 6075 6175 20  0000 C CNN
-F 2 "MX_Alps_Hybrid:MXOnly-1.25U" H 6050 6100 60  0001 C CNN
+F 0 "SW_LALT1" H 6075 6250 60  0000 C CNN
+F 1 "1.25U" H 6075 6175 20  0000 C CNN
+F 2 "MX_Alps_Hybrid:MX-1.25U" H 6050 6100 60  0001 C CNN
 F 3 "" H 6050 6100 60  0001 C CNN
 	1    6075 6125
@@
 $EndComp
 $Comp
-L MX_Alps_Hybrids:MX-6.25U MX_SP1
+L MX_Alps_Hybrids:MX-6.25U SW_SP1
 U 1 1 5A2F4C87
 P 8575 6125
-F 0 "MX_SP1" H 8575 6250 60  0000 C CNN
-F 1 "MX-6.25U" H 8575 6175 20  0000 C CNN
-F 2 "MX_Alps_Hybrid:MXOnly-6.25U-ReversedStabilizers" H 8550 6100 60  0001 C CNN
+F 0 "SW_SP1" H 8575 6250 60  0000 C CNN
+F 1 "6.25U" H 8575 6175 20  0000 C CNN
+F 2 "MX_Alps_Hybrid:MX-6.25U-ReversedStabilizers" H 8550 6100 60  0001 C CNN
 F 3 "" H 8550 6100 60  0001 C CNN
 	1    8575 6125
@@
 $EndComp
 $Comp
-L MX_Alps_Hybrids:MX-1.25U MX_RALT1
+L MX_Alps_Hybrids:MX-1.25U SW_RALT1
 U 1 1 5A2F4D13
 P 11075 6125
-F 0 "MX_RALT1" H 11075 6250 60  0000 C CNN
-F 1 "MX-1.25U" H 11075 6175 20  0000 C CNN
-F 2 "MX_Alps_Hybrid:MXOnly-1.25U" H 11050 6100 60  0001 C CNN
+F 0 "SW_RALT1" H 11075 6250 60  0000 C CNN
+F 1 "1.25U" H 11075 6175 20  0000 C CNN
+F 2 "MX_Alps_Hybrid:MX-1.25U" H 11050 6100 60  0001 C CNN
 F 3 "" H 11050 6100 60  0001 C CNN
 	1    11075 6125
@@
 $EndComp
 $Comp
-L MX_Alps_Hybrids:MX-1.25U MX_RGUI1
+L MX_Alps_Hybrids:MX-1.25U SW_RGUI1
 U 1 1 5A2F4D27
 P 11700 6125
-F 0 "MX_RGUI1" H 11700 6250 60  0000 C CNN
-F 1 "MX-1.25U" H 11700 6175 20  0000 C CNN
-F 2 "MX_Alps_Hybrid:MXOnly-1.25U-FLIPPED" H 11675 6100 60  0001 C CNN
+F 0 "SW_RGUI1" H 11700 6250 60  0000 C CNN
+F 1 "1.25U" H 11700 6175 20  0000 C CNN
+F 2 "MX_Alps_Hybrid:MX-1.25U-FLIPPED" H 11675 6100 60  0001 C CNN
 F 3 "" H 11675 6100 60  0001 C CNN
 	1    11700 6125
@@
 $EndComp
 $Comp
-L MX_Alps_Hybrids:MX-1.5U MX_LCTRL2
+L MX_Alps_Hybrids:MX-1.5U SW_LCTRL2
 U 1 1 5A33B842
 P 4825 6800
-F 0 "MX_LCTRL2" H 4825 6925 60  0000 C CNN
-F 1 "MX-1.5U" H 4825 6850 20  0000 C CNN
-F 2 "MX_Alps_Hybrid:MXOnly-1.5U-FLIPPED" H 4800 6775 60  0001 C CNN
+F 0 "SW_LCTRL2" H 4825 6925 60  0000 C CNN
+F 1 "1.5U" H 4825 6850 20  0000 C CNN
+F 2 "MX_Alps_Hybrid:MX-1.5U-FLIPPED" H 4800 6775 60  0001 C CNN
 F 3 "" H 4800 6775 60  0001 C CNN
 	1    4825 6800
@@
 $EndComp
 $Comp
-L MX_Alps_Hybrids:MX-1.5U MX_LGUI2
+L MX_Alps_Hybrids:MX-1.5U SW_LGUI2
 U 1 1 5A33B86A
 P 5450 6800
-F 0 "MX_LGUI2" H 5450 6925 60  0000 C CNN
-F 1 "MX-1U" H 5450 6850 20  0000 C CNN
-F 2 "MX_Alps_Hybrid:MXOnly-1U-FLIPPED" H 5425 6775 60  0001 C CNN
+F 0 "SW_LGUI2" H 5450 6925 60  0000 C CNN
+F 1 "1U" H 5450 6850 20  0000 C CNN
+F 2 "MX_Alps_Hybrid:MX-1U-FLIPPED" H 5425 6775 60  0001 C CNN
 F 3 "" H 5425 6775 60  0001 C CNN
 	1    5450 6800
@@
 $EndComp
 $Comp
-L MX_Alps_Hybrids:MX-1.5U MX_RALT2
+L MX_Alps_Hybrids:MX-1.5U SW_RALT2
 U 1 1 5A33B95A
 P 11700 6800
-F 0 "MX_RALT2" H 11700 6925 60  0000 C CNN
-F 1 "MX-1.5U" H 11700 6850 20  0000 C CNN
-F 2 "MX_Alps_Hybrid:MXOnly-1.5U" H 11675 6775 60  0001 C CNN
+F 0 "SW_RALT2" H 11700 6925 60  0000 C CNN
+F 1 "1.5U" H 11700 6850 20  0000 C CNN
+F 2 "MX_Alps_Hybrid:MX-1.5U" H 11675 6775 60  0001 C CNN
 F 3 "" H 11675 6775 60  0001 C CNN
 	1    11700 6800
@@
 $EndComp
 $Comp
-L MX_Alps_Hybrids:MX-1U MX_RCTRL1
+L MX_Alps_Hybrids:MX-1U SW_RCTRL1
 U 1 1 5A2F4D4F
 P 12950 6125
-F 0 "MX_RCTRL1" H 12950 6250 60  0000 C CNN
-F 1 "MX-1.25U" H 12950 6175 20  0000 C CNN
-F 2 "MX_Alps_Hybrid:MXOnly-1.25U-FLIPPED" H 12925 6100 60  0001 C CNN
+F 0 "SW_RCTRL1" H 12950 6250 60  0000 C CNN
+F 1 "1.25U" H 12950 6175 20  0000 C CNN
+F 2 "MX_Alps_Hybrid:MX-1.25U-FLIPPED" H 12925 6100 60  0001 C CNN
 F 3 "" H 12925 6100 60  0001 C CNN
 	1    12950 6125
@@
 $EndComp
 $Comp
-L MX_Alps_Hybrids:MX-1U MX_RMENU1
+L MX_Alps_Hybrids:MX-1U SW_RMENU1
 U 1 1 5A2F4D3B
 P 12325 6125
-F 0 "MX_RMENU1" H 12325 6250 60  0000 C CNN
+F 0 "SW_RMENU1" H 12325 6250 60  0000 C CNN
 F 1 "MX-1.25U" H 12325 6175 20  0000 C CNN
-F 2 "MX_Alps_Hybrid:MXOnly-1.25U-FLIPPED" H 12300 6100 60  0001 C CNN
+F 2 "MX_Alps_Hybrid:MX-1.25U-FLIPPED" H 12300 6100 60  0001 C CNN
 F 3 "" H 12300 6100 60  0001 C CNN
 	1    12325 6125
@@
 $EndComp
 $Comp
-L MX_Alps_Hybrids:MX-1U MX_RT1
+L MX_Alps_Hybrids:MX-1U SW_RT1
 U 1 1 5ADD1F97
 P 16825 6125
-F 0 "MX_RT1" H 16825 6250 60  0000 C CNN
-F 1 "MX-1U" H 16825 6175 20  0000 C CNN
-F 2 "MX_Alps_Hybrid:MXOnly-1U" H 16800 6100 60  0001 C CNN
+F 0 "SW_RT1" H 16825 6250 60  0000 C CNN
+F 1 "1U" H 16825 6175 20  0000 C CNN
+F 2 "MX_Alps_Hybrid:MX-1U" H 16800 6100 60  0001 C CNN
 F 3 "" H 16800 6100 60  0001 C CNN
 	1    16825 6125
@@
 $EndComp
 $Comp
-L MX_Alps_Hybrids:MX-1U MX_DN1
+L MX_Alps_Hybrids:MX-1U SW_DN1
 U 1 1 5ADD1F85
 P 16200 6125
-F 0 "MX_DN1" H 16200 6250 60  0000 C CNN
-F 1 "MX-1U" H 16200 6175 20  0000 C CNN
-F 2 "MX_Alps_Hybrid:MXOnly-1U" H 16175 6100 60  0001 C CNN
+F 0 "SW_DN1" H 16200 6250 60  0000 C CNN
+F 1 "1U" H 16200 6175 20  0000 C CNN
+F 2 "MX_Alps_Hybrid:MX-1U" H 16175 6100 60  0001 C CNN
 F 3 "" H 16175 6100 60  0001 C CNN
 	1    16200 6125
@@
 $EndComp
 $Comp
-L MX_Alps_Hybrids:MX-1U MX_LFT1
+L MX_Alps_Hybrids:MX-1U SW_LFT1
 U 1 1 5ADD1F73
 P 15575 6125
-F 0 "MX_LFT1" H 15575 6250 60  0000 C CNN
-F 1 "MX-1U" H 15575 6175 20  0000 C CNN
-F 2 "MX_Alps_Hybrid:MXOnly-1U" H 15550 6100 60  0001 C CNN
+F 0 "SW_LFT1" H 15575 6250 60  0000 C CNN
+F 1 "1U" H 15575 6175 20  0000 C CNN
+F 2 "MX_Alps_Hybrid:MX-1U" H 15550 6100 60  0001 C CNN
 F 3 "" H 15550 6100 60  0001 C CNN
 	1    15575 6125
@@
 $EndComp
 $Comp
-L MX_Alps_Hybrids:MX-1.5U MX_LALT2
+L MX_Alps_Hybrids:MX-1.5U SW_LALT2
 U 1 1 5DF0F6D0
 P 6075 6800
-F 0 "MX_LALT2" H 6075 6925 60  0000 C CNN
-F 1 "MX-1.5U" H 6075 6850 20  0000 C CNN
-F 2 "MX_Alps_Hybrid:MXOnly-1.5U-FLIPPED" H 6050 6775 60  0001 C CNN
+F 0 "SW_LALT2" H 6075 6925 60  0000 C CNN
+F 1 "1.5U" H 6075 6850 20  0000 C CNN
+F 2 "MX_Alps_Hybrid:MX-1.5U-FLIPPED" H 6050 6775 60  0001 C CNN
 F 3 "" H 6050 6775 60  0001 C CNN
 	1    6075 6800
@@
 Connection ~ 11200 5475
 $Comp
-L MX_Alps_Hybrids:MX-1.5U MX_RGUI2
+L MX_Alps_Hybrids:MX-1.5U SW_RGUI2
 U 1 1 5EF309B7
 P 12325 6800
-F 0 "MX_RGUI2" H 12325 6925 60  0000 C CNN
-F 1 "MX-1U" H 12325 6850 20  0000 C CNN
-F 2 "MX_Alps_Hybrid:MXOnly-1U" H 12300 6775 60  0001 C CNN
+F 0 "SW_RGUI2" H 12325 6925 60  0000 C CNN
+F 1 "1U" H 12325 6850 20  0000 C CNN
+F 2 "MX_Alps_Hybrid:MX-1U" H 12300 6775 60  0001 C CNN
 F 3 "" H 12300 6775 60  0001 C CNN
 	1    12325 6800
@@
 $EndComp
 $Comp
-L MX_Alps_Hybrids:MX-1.5U MX_RCTRL2
+L MX_Alps_Hybrids:MX-1.5U SW_RCTRL2
 U 1 1 5EF3106A
 P 12950 6800
-F 0 "MX_RCTRL2" H 12950 6925 60  0000 C CNN
-F 1 "MX-1.5U" H 12950 6850 20  0000 C CNN
-F 2 "MX_Alps_Hybrid:MXOnly-1.5U" H 12925 6775 60  0001 C CNN
+F 0 "SW_RCTRL2" H 12950 6925 60  0000 C CNN
+F 1 "1.5U" H 12950 6850 20  0000 C CNN
+F 2 "MX_Alps_Hybrid:MX-1.5U" H 12925 6775 60  0001 C CNN
 F 3 "" H 12925 6775 60  0001 C CNN
 	1    12950 6800
@@
 Connection ~ 5425 6300
 $Comp
-L MX_Alps_Hybrids:MX-7U MX_SP2
+L MX_Alps_Hybrids:MX-7U SW_SP2
 U 1 1 5A33B8BA
 P 8575 6800
-F 0 "MX_SP2" H 8575 6925 60  0000 C CNN
-F 1 "MX-7U" H 8575 6850 20  0000 C CNN
-F 2 "MX_Alps_Hybrid:MXOnly-7U-ReversedStabilizers" H 8550 6775 60  0001 C CNN
+F 0 "SW_SP2" H 8575 6925 60  0000 C CNN
+F 1 "7U" H 8575 6850 20  0000 C CNN
+F 2 "MX_Alps_Hybrid:MX-7U-ReversedStabilizers" H 8550 6775 60  0001 C CNN
 F 3 "" H 8550 6775 60  0001 C CNN
 	1    8575 6800
